File: PCB/gb_walkie.sch (KiCad schematic (older format))
At the start: 71 parts, among them J1 USB_OTG, J2 HPJACK, J3 Micro_SD_Card, SW1 Rotary_Encoder_Switch, SW2 SW_Push, SW3 SW_Push, SW5 POWER, SW6 SW_DIP_x03, U1 SAMD21_MOD, U2 CODECODER-VS1053B(LQFP48)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

Commit message: updated component part number
Parts:
- C16: Digikey Part No. 311-1729-1-ND -> 1276-6456-1-ND
Changed lines of the file:
@@
 F 2 "Capacitor_SMD:C_0805_2012Metric" H 12500 3550 50  0001 C CNN
 F 3 "~" H 12500 3550 50  0001 C CNN
-F 4 "311-1729-1-ND" H 12500 3550 50  0001 C CNN "Digikey Part No."
+F 4 "1276-6456-1-ND" H 12500 3550 50  0001 C CNN "Digikey Part No."
 	1    12500 3550
 	-1   0    0    1
